File: ermatic_mini.kicad_pcb (KiCad board)
At the start: 2 copper layers, 100 x 100 mm, 62 parts, among them J1 GND, J10 R1, J13 LOW, J2 VIN, J21 AC, J22 GPIO, J23 USB_B, J24 UART, J4 R1, J5 LOW, J6 R1, J7 LOW, J8 R1, J9 LOW, SW1 !EN, SW3 !GPIO9, U1 ESP32-C6-WROOM-1, U2 LDI1117-3.3H-DIO, U3 LTV-847, U6 LDI1117-3.3H-DIO, U7 LDI1117-05H-DIO

Commit message: first bugs fixed
Parts:
- added D2: BZV55C2V7, Diode_SMD:D_MiniMELF, F.Cu at (129.4, 60.8)
- added J11: BUZZER, Connector_PinHeader_1.27mm:PinHeader_1x02_P1.27mm_Vertical, F.Cu at (112.2, 81.8)
- added J3: GP2x, Connector_PinHeader_1.27mm:PinHeader_1x04_P1.27mm_Vertical, F.Cu at (119.2, 104.0)
- R23: value 360 -> 100
- moved R23 6.35 mm to (124.3, 60.8)
Connections:
- D20 pad 2: Net-(D20-A) -> Net-(D2-A)
- R23 pad 2: Net-(D20-A) -> Net-(D2-K)
Routing:
- net GPIO10: track 0.00 -> 10.4 mm
- net GND: track 478.3 -> 483.6 mm
- net Net-(D2-A): track 0.00 -> 4.47 mm
- net USB_PWR: track 33.1 -> 29.2 mm
- net Net-(D20-A): track 3.49 -> 0.00 mm
- net GPIO22: track 0.00 -> 2.05 mm
- net GPIO23: track 0.00 -> 2.05 mm
- net GPIO21: track 0.00 -> 2.05 mm
- net GPIO20: track 0.00 -> 2.05 mm
- net Net-(D2-K): track 0.00 -> 1.87 mm
- net USBD-: track 14.9 -> 16.6 mm
- net +3V3: track 265.5 -> 264.1 mm
- net EN: track 56.1 -> 57.1 mm
- net GPIO8: track 19.6 -> 20.1 mm
Other:
- board text added: "(10)"
- board text added: "(20-23)"
- board text added: "(5)"
- board text added: "(6)"
- board text added: "(7)"
- board text added: "BOOT"
- board text added: "EN"
