File: ermatic_mini.kicad_sch (KiCad schematic)
At the start: 37 parts, among them J1 GND, J2 VIN, J21 AC, J22 GPIO, J23 USB_B, J24 UART, SW1 !EN, SW3 !GPIO9, U1 ESP32-C6-WROOM-1, U2 LDI1117-3.3H-DIO, U6 LDI1117-3.3H-DIO, U7 LDI1117-05H-DIO

Commit message: first bugs fixed
Parts:
- added D12, D14, D16, D3: BAT760, Diode_SMD:D_SOD-323_HandSoldering, symbol Diode:BAT85
- added D2: BZV55C2V7, Diode_SMD:D_MiniMELF, symbol Device:D_Zener
- added J10, J4, J6, J8: R1, TerminalBlock_4Ucon:TerminalBlock_4Ucon_1x03_P3.50mm_Horizontal, symbol Connector:Screw_Terminal_01x03
- added J11: BUZZER, Connector_PinHeader_1.27mm:PinHeader_1x02_P1.27mm_Vertical, symbol Connector:Conn_01x02_Pin
- added J13, J5, J7, J9: LOW, Connector_Pin:Pin_D1.0mm_L10.0mm, symbol Connector:Conn_01x01_Socket
- added J3: GP2x, Connector_PinHeader_1.27mm:PinHeader_1x04_P1.27mm_Vertical, symbol Connector:Conn_01x04_Pin
- added JP1, JP2, JP3, JP4: GND, Jumper:SolderJumper-2_P1.3mm_Open_TrianglePad1.0x1.5mm, symbol Jumper:Jumper_2_Small_Bridged
- added R18, R26, R31, R7: 100, Resistor_SMD:R_1206_3216Metric, symbol Device:R_Small
- added RL1, RL2, RL3, RL4: (no value), jb_missing:RM87N, symbol jb_missing:RM87N
- added U3: LTV-847, Package_DIP:DIP-16_W7.62mm, symbol Isolator:LTV-847
- R23: value 360 -> 100
Connections:
- net +12V: now also D12.1 (K), D14.1 (K), D16.1 (K), D3.1 (K), RL1.A1, RL2.A1, RL3.A1, RL4.A1
- net GND: now also J11.2 (Pin_2), JP1.2 (B), JP2.2 (B), JP3.2 (B), JP4.2 (B), U3.2, U3.4, U3.6, U3.8
- net GPIO10: now also J11.1 (Pin_1)
- net GPIO11: now also R7.1
- net GPIO15: now also R18.1
- net GPIO18: now also R26.1
- net GPIO19: now also R31.1
- net GPIO20: now also J3.1 (Pin_1)
- net GPIO21: now also J3.2 (Pin_2)
- net GPIO22: now also J3.3 (Pin_3)
- net GPIO23: now also J3.4 (Pin_4)
- net at R23.2: now also D2.1 (K); no longer D20.2 (A)
- new net: D16.2 (A), RL4.A2, U3.16
- new net: J13.1 (Pin_1), JP4.1 (A), U3.15
- new net: R31.2, U3.1
- new net: D12.2 (A), RL2.A2, U3.12
- new net: J4.3 (Pin_3), RL1.11
- new net: J4.2 (Pin_2), RL1.12
- new net: J4.1 (Pin_1), RL1.14
- new net: D3.2 (A), RL1.A2, U3.10
- new net: J9.1 (Pin_1), JP3.1 (A), U3.13
- new net: R7.2, U3.7
- new net: J5.1 (Pin_1), JP1.1 (A), U3.9
- new net: J7.1 (Pin_1), JP2.1 (A), U3.11
- new net: R26.2, U3.3
- new net: J6.3 (Pin_3), RL2.11
- new net: J6.2 (Pin_2), RL2.12
- new net: J6.1 (Pin_1), RL2.14
- new net: J8.3 (Pin_3), RL3.11
- new net: J8.2 (Pin_2), RL3.12
- new net: J8.1 (Pin_1), RL3.14
- new net: D14.2 (A), RL3.A2, U3.14
- new net: R18.2, U3.5
- new net: D2.2 (A), D20.2 (A)
- new net: J10.1 (Pin_1), RL4.14
- new net: J10.2 (Pin_2), RL4.12
- new net: J10.3 (Pin_3), RL4.11
Other:
- removed sheet executive-part
- moved on the sheet: C10, C13, C6, C8, D20, F1, F2, F3, J21, J23, L3, PS1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
